File: tako_assembled/pcb/tako.kicad_sch (KiCad schematic)
At the start: 144 parts, among them J1 MJ-4PP-9, J101 MJ-4PP-9, SW1 EC_SW, SW10 EC_SW, SW11 EC_SW, SW12 EC_SW, SW13 EC_SW, SW14 EC_SW, SW15 EC_SW, SW2 EC_SW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

Commit message: Get rid of old name
Other:
- title: Thocktopus -> tako
