File: rev1/pcb/tako.kicad_pcb (KiCad board)
At the start: 2 copper layers, 230.7 x 97.8 mm, 120 parts, among them J1 MJ-4PP-9, J101 MJ-4PP-9, SW1 EC_SW, SW10 EC_SW, SW101 EC_SW, SW102 EC_SW, SW103 EC_SW, SW104 EC_SW, SW105 EC_SW, SW106 EC_SW, SW107 EC_SW, SW108 EC_SW, SW109 EC_SW, SW11 EC_SW, SW110 EC_SW, SW111 EC_SW, SW112 EC_SW, SW113 EC_SW, SW114 EC_SW, SW115 EC_SW, SW116 EC_SW, SW117 EC_SW, SW12 EC_SW, SW13 EC_SW, SW14 EC_SW, SW15 EC_SW, SW16 EC_SW, SW17 EC_SW, SW2 EC_SW, SW3 EC_SW, SW4 EC_SW, SW5 EC_SW, SW6 EC_SW, SW7 EC_SW, SW8 EC_SW, SW9 EC_SW, U1 STeMCell, U101 STeMCell, U102 74HC4051, U103 OPA350, U2 74HC4051, U3 OPA350

Commit message: updated code for 36key
Parts:
- added H18: MountingHole, tako:MountingHole_3.4mm, F.Cu at (45.8, 116.7)
- added H19: MountingHole, tako:MountingHole_3.4mm, F.Cu at (257.7, 116.7)
- added SW118: EC_SW, tako:ecs_pad_1U_no_ring_90deg, F.Cu at (74.6, 103.3)
- added SW18: EC_SW, tako:ecs_pad_1U_no_ring_90deg, F.Cu at (228.9, 103.3)
- moved H14 35.3 mm to (274.7, 117.0)
- moved SW17 35.2 mm to (248.7, 111.5), turned to 150 degrees
- moved SW16 33.9 mm to (265.2, 124.0), turned to 135 degrees
- moved RSW1 17.5 mm to (265.1, 105.4), turned to -90 degrees
- moved R106 16.8 mm to (124.1, 100.0)
- moved H114 16.6 mm to (28.9, 117.0)
- moved R105 16.2 mm to (127.4, 104.0)
- moved J1 15.6 mm to (266.7, 97.0)
- moved SW116 15.3 mm to (38.3, 124.0), turned to -135 degrees
- moved SW104 14.1 mm to (83.8, 43.4)
- moved JP1 14.1 mm to (207.6, 95.9)
- moved SW110 14.1 mm to (64.7, 64.9)
- moved mouse-bite-2mm-slot 14.1 mm to (151.8, 83.7)
- moved H103 14.1 mm to (140.9, 83.4)
- moved R108 14.1 mm to (120.4, 95.6)
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Routing:
- net COL2_R: track 102.9 -> 163.7 mm, vias 3 -> 6
- net COL2: track 106.0 -> 160.6 mm, vias 3 -> 6
- net COL1_R: track 155.7 -> 186.9 mm
- net COL0_R: track 170.7 -> 197.8 mm
- net COL1: track 160.0 -> 185.7 mm
- net Net-(R4-Pad2): track 27.0 -> 52.3 mm, vias 3 -> 4
- net Net-(R104-Pad2): track 26.7 -> 51.2 mm, vias 3 -> 4
- net COL0: track 169.9 -> 193.9 mm
- net RESET: track 53.1 -> 56.6 mm
- net RESET_R: track 42.8 -> 45.6 mm
- net GND_R: track 0.00 -> 2.54 mm, vias 102 -> 111
- net DATA: track 43.6 -> 44.7 mm
- net +3.3V: track 51.6 -> 52.6 mm
- net DATA_R: track 42.2 -> 42.9 mm
- net +3.3V_R: track 37.7 -> 37.2 mm
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Other:
- board size 230.7 x 97.8 mm -> 252.1 x 110.4 mm
