File: rev1/plates/bottom/bottom_plate.kicad_pcb (KiCad board)
At the start: 2 copper layers, 114 x 97.8 mm, 20 parts, among them J1 MJ-4PP-9, U1 STeMCell

Commit message: updated code for 36key
Parts:
- removed DISP1: nice!view, tako:nice_view_cutout
- removed H1, H10, H11, H12, H13, H14, H2, H3, H4, H5, H6, H7, H8, H9: MountingHole, tako:M2_hole_4.2mm
- removed H15 (x2), H16: MountingHole, tako:M2_hole_3.5mm
- removed J1: MJ-4PP-9, tako:TRRS-PJ-320A_cutout
- removed U1: STeMCell, tako:ArduinoProMicro_cutout
- added DISP101: nice!view, tako:nice_view_cutout, F.Cu at (45.8, 75.9)
- added H101: MountingHole, tako:M2_hole_4.2mm, F.Cu at (140.9, 44.7)
- added H102: MountingHole, tako:M2_hole_4.2mm, F.Cu at (140.9, 64.4)
- added H103: MountingHole, tako:M2_hole_4.2mm, F.Cu at (140.9, 83.4)
- added H104: MountingHole, tako:M2_hole_4.2mm, F.Cu at (121.9, 32.7)
- added H105: MountingHole, tako:M2_hole_4.2mm, F.Cu at (126.9, 95.0)
- added H106: MountingHole, tako:M2_hole_4.2mm, F.Cu at (102.8, 46.4)
- added H107: MountingHole, tako:M2_hole_4.2mm, F.Cu at (102.8, 65.4)
- added H108: MountingHole, tako:M2_hole_4.2mm, F.Cu at (102.8, 87.0)
- added H109: MountingHole, tako:M2_hole_4.2mm, F.Cu at (83.8, 33.2)
- added H110: MountingHole, tako:M2_hole_4.2mm, F.Cu at (64.7, 35.7)
- added H111: MountingHole, tako:M2_hole_4.2mm, F.Cu at (64.7, 55.4)
- added H112: MountingHole, tako:M2_hole_4.2mm, F.Cu at (64.7, 74.4)
- added H113: MountingHole, tako:M2_hole_4.2mm, F.Cu at (64.2, 106.2)
- added H114: MountingHole, tako:M2_hole_4.2mm, F.Cu at (28.9, 117.0)
- added H115: MountingHole, tako:M2_hole_3.5mm, F.Cu at (53.2, 54.5)
- added H116: MountingHole, tako:M2_hole_3.5mm, F.Cu at (38.4, 54.5)
- added H18: MountingHole, tako:M2_hole_4.2mm, F.Cu at (45.8, 116.7)
- added J101: MJ-4PP-9, tako:TRRS-PJ-320A_cutout, F.Cu at (36.7, 97.0)
- added L1: ART, personal-logo:peacock-large, B.Cu at (102.6, 80.5)
- added L2: ART, personal-logo:peacock-large, F.Cu at (100.7, 81.4)
- added U101: STeMCell, tako:ArduinoProMicro_cutout, B.Cu at (45.8, 74.3)
Routing:
- added copper zone on B.Cu, net GND_R
- added copper zone on F.Cu, net GND_R
Other:
- board size 114 x 97.8 mm -> 124.7 x 110.4 mm
