File: rev1/plates/top/niz/top_plate_niz.kicad_pcb (KiCad board)
At the start: 2 copper layers, 111.7 x 97.8 mm, 32 parts, among them SW1 EC_SW, SW10 EC_SW, SW11 EC_SW, SW12 EC_SW, SW13 EC_SW, SW14 EC_SW, SW15 EC_SW, SW16 EC_SW, SW17 EC_SW, SW2 EC_SW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

Commit message: updated code for 36key
Parts:
- removed G***: LOGO, tako:tako
- removed H1, H10, H11, H12, H13, H14, H2, H3, H4, H5, H6, H7, H8, H9: MountingHole, tako:M2_hole_4.2mm
- removed SW1, SW10, SW11, SW12, SW13, SW14, SW15, SW16, SW17, SW2, SW3, SW4, SW5, SW6, SW7, SW8, SW9: EC_SW, tako:plate_cut_ecs_pad_NIZ
- added H101: MountingHole, tako:M2_hole_4.2mm, F.Cu at (140.9, 44.7)
- added H102: MountingHole, tako:M2_hole_4.2mm, F.Cu at (140.9, 64.4)
- added H103: MountingHole, tako:M2_hole_4.2mm, F.Cu at (140.9, 83.4)
- added H104: MountingHole, tako:M2_hole_4.2mm, F.Cu at (121.9, 32.7)
- added H105: MountingHole, tako:M2_hole_4.2mm, F.Cu at (126.9, 95.0)
- added H106: MountingHole, tako:M2_hole_4.2mm, F.Cu at (102.8, 46.4)
- added H107: MountingHole, tako:M2_hole_4.2mm, F.Cu at (102.8, 65.4)
- added H108: MountingHole, tako:M2_hole_4.2mm, F.Cu at (102.8, 87.0)
- added H109: MountingHole, tako:M2_hole_4.2mm, F.Cu at (83.8, 33.2)
- added H110: MountingHole, tako:M2_hole_4.2mm, F.Cu at (64.7, 35.7)
- added H111: MountingHole, tako:M2_hole_4.2mm, F.Cu at (64.7, 55.4)
- added H112: MountingHole, tako:M2_hole_4.2mm, F.Cu at (64.7, 74.4)
- added H113: MountingHole, tako:M2_hole_4.2mm, F.Cu at (64.2, 106.2)
- added H114: MountingHole, tako:M2_hole_4.2mm, F.Cu at (28.9, 117.0)
- added H18: MountingHole, tako:M2_hole_4.2mm, F.Cu at (45.8, 116.7)
- added L1: Art, personal-logo:peacock-medium, F.Cu at (110.8, 97.7)
- added L2: Art, personal-logo:peacock-medium, B.Cu at (108.6, 98.5)
- added SW101: EC_SW, tako:plate_cut_ecs_pad_NIZ, F.Cu at (140.9, 54.9)
- added SW102: EC_SW, tako:plate_cut_ecs_pad_NIZ, F.Cu at (121.9, 42.9)
- added SW103: EC_SW, tako:plate_cut_ecs_pad_NIZ, F.Cu at (102.8, 36.9)
- added SW104: EC_SW, tako:plate_cut_ecs_pad_NIZ, F.Cu at (83.8, 43.4)
- added SW105: EC_SW, tako:plate_cut_ecs_pad_NIZ, F.Cu at (64.7, 45.9)
- added SW106: EC_SW, tako:plate_cut_ecs_pad_NIZ, F.Cu at (140.9, 73.9)
- added SW107: EC_SW, tako:plate_cut_ecs_pad_NIZ, F.Cu at (121.9, 61.9)
- added SW108: EC_SW, tako:plate_cut_ecs_pad_NIZ, F.Cu at (102.8, 55.9)
- added SW109: EC_SW, tako:plate_cut_ecs_pad_NIZ, F.Cu at (83.8, 62.4)
- added SW110: EC_SW, tako:plate_cut_ecs_pad_NIZ, F.Cu at (64.7, 64.9)
- added SW111: EC_SW, tako:plate_cut_ecs_pad_NIZ, F.Cu at (140.9, 93.0)
- added SW112: EC_SW, tako:plate_cut_ecs_pad_NIZ, F.Cu at (121.9, 81.0)
- added SW113: EC_SW, tako:plate_cut_ecs_pad_NIZ, F.Cu at (102.8, 75.0)
- added SW114: EC_SW, tako:plate_cut_ecs_pad_NIZ, F.Cu at (83.8, 81.5)
- added SW115: EC_SW, tako:plate_cut_ecs_pad_NIZ, F.Cu at (64.7, 84.0)
- added SW116: EC_SW, tako:plate_cut_ecs_pad_NIZ, F.Cu at (38.3, 124.0)
- added SW117: EC_SW, tako:plate_cut_ecs_pad_NIZ, F.Cu at (54.9, 111.5)
- added SW118: EC_SW, tako:plate_cut_ecs_pad_NIZ, F.Cu at (74.6, 103.3)
Routing:
- added copper zone on B.Cu, net GND_R
- added copper zone on F.Cu, net GND_R
Other:
- board size 111.7 x 97.8 mm -> 124.7 x 110.4 mm
- board text added: "TAKO 36 REV 1.0 BY SSBB MOD HarshitGoel96"
